File: kicad/pi-pic-proto-hat/pipicproto.kicad_pcb (KiCad board)
At the start: 2 copper layers, 65 x 56 mm, 5 parts, among them P1 Conn_02x20_Odd_Even

Commit message: version-b
Parts:
- added C1: 100n, Capacitor_THT:C_Disc_D3.8mm_W2.6mm_P2.50mm, F.Cu at (259.1, 119.5)
- added D1: D_Schottky, Diode_THT:D_A-405_P7.62mm_Horizontal, F.Cu at (254.6, 105.5)
- added J1: Conn_01x02_Male, Connector_PinHeader_2.54mm:PinHeader_1x02_P2.54mm_Vertical, F.Cu at (207.6, 141.1)
- added J10: Conn_01x13_Male, Connector_PinHeader_2.54mm:PinHeader_1x13_P2.54mm_Vertical, F.Cu at (203.8, 134.8)
- added J2: Conn_01x02_Male, Connector_Phoenix_MC:PhoenixContact_MC_1,5_2-G-3.81_1x02_P3.81mm_Horizontal, F.Cu at (238.1, 142.4)
- added J22: Conn_01x13_Male, Connector_PinHeader_2.54mm:PinHeader_1x13_P2.54mm_Vertical, F.Cu at (203.8, 106.8)
- added J3: Conn_01x02_Male, Connector_Phoenix_MC:PhoenixContact_MC_1,5_2-G-3.81_1x02_P3.81mm_Horizontal, F.Cu at (214.0, 142.4)
- added J4: Conn_01x02_Male, Connector_PinHeader_2.54mm:PinHeader_1x02_P2.54mm_Vertical, F.Cu at (241.9, 136.0)
- added J5: Conn_01x02_Male, Connector_PinHeader_2.54mm:PinHeader_1x02_P2.54mm_Vertical, F.Cu at (241.9, 132.2)
- added J6: Barrel_Jack_Switch, Connector_BarrelJack:BarrelJack_CUI_PJ-102AH_Horizontal, F.Cu at (250.8, 136.4)
- added J7: Conn_01x20_Male, Connector_PinHeader_2.54mm:PinHeader_1x20_P2.54mm_Vertical, F.Cu at (203.8, 103.0)
- added J8: Conn_01x06_Male, Connector_PinHeader_2.54mm:PinHeader_1x06_P2.54mm_Vertical, F.Cu at (262.2, 114.4)
- added J9: Conn_01x06_Male, Connector_PinHeader_2.54mm:PinHeader_1x06_P2.54mm_Vertical, F.Cu at (238.1, 114.4)
- added Q1: IRF4905, Package_TO_SOT_THT:TO-220-3_Vertical, F.Cu at (225.4, 147.5)
- added R1: 10k, Resistor_THT:R_Axial_DIN0207_L6.3mm_D2.5mm_P10.16mm_Horizontal, F.Cu at (233.0, 141.1)
- added R2: 1k, Resistor_THT:R_Axial_DIN0207_L6.3mm_D2.5mm_P10.16mm_Horizontal, F.Cu at (222.9, 138.6)
- added R3: 1k, Resistor_THT:R_Axial_DIN0207_L6.3mm_D2.5mm_P10.16mm_Horizontal, F.Cu at (258.4, 114.4)
- added R4: 22k, Resistor_THT:R_Axial_DIN0207_L6.3mm_D2.5mm_P10.16mm_Horizontal, F.Cu at (262.2, 109.4)
- added R5: 1k, Resistor_THT:R_Axial_DIN0207_L6.3mm_D2.5mm_P10.16mm_Horizontal, F.Cu at (241.3, 125.9)
- added R6: 1k, Resistor_THT:R_Axial_DIN0207_L6.3mm_D2.5mm_P10.16mm_Horizontal, F.Cu at (244.4, 127.1)
- added REF**: Lora_3x5, myfootprint:Lora_3x5, F.Cu at (231.8, 119.5)
- added REF**: Lora_3x5, myfootprint:Lora_3x5, F.Cu at (231.8, 106.8)
- added REF**: Lora_5x5, myfootprint:Lora_5x5, F.Cu at (221.6, 119.5)
- added REF**: Lora_5x5, myfootprint:Lora_5x5, F.Cu at (208.9, 119.5)
- added REF**: Lora_5x5, myfootprint:Lora_5x5, F.Cu at (221.6, 106.8)
- added REF**: Lora_5x5, myfootprint:Lora_5x5, F.Cu at (208.9, 106.8)
- added SW1: SW_Push, Button_Switch_THT:SW_PUSH_6mm_H9.5mm, F.Cu at (248.3, 110.6)
- added U1: PIC12F675-IP, Package_DIP:DIP-8_W7.62mm, F.Cu at (255.9, 118.2)
- renumbered MK3 to MK2, MK2 to MK3
Routing:
- net +5V: track 0.00 -> 83.0 mm
- net +5VP: track 0.00 -> 69.1 mm
- net /GPIO25(GEN6): track 0.00 -> 53.1 mm
- net +3V3: track 0.00 -> 33.2 mm
- net Net-(J1-Pad1): track 0.00 -> 31.9 mm
- net /IO2: track 0.00 -> 27.4 mm
- net /DAT: track 0.00 -> 26.5 mm
- net /GPIO7(SPI1_CE_N): track 0.00 -> 23.1 mm
- net /CLK: track 0.00 -> 22.9 mm
- net /MCLR: track 0.00 -> 21.7 mm
- net /IO5: track 0.00 -> 18.9 mm
- net /GPIO8(SPI0_CE_N): track 0.00 -> 17.8 mm
- net /IO4: track 0.00 -> 15.3 mm
- net /GPIO10(SPI0_MOSI): track 0.00 -> 12.4 mm
- net /GPIO11(SPI0_SCK): track 0.00 -> 12.4 mm
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Other:
- outline, holes or cut-outs redrawn

Commit message: version-d
Routing:
- net +5VP: track 69.1 -> 84.7 mm
- net /IO2: track 27.4 -> 12.8 mm
- net /MCLR: track 21.7 -> 20.6 mm
- added copper zone on B.Cu, net GND
Other:
- board text added: "+3V3"
- board text added: "+5V"
- board text added: "-"
- board text added: "0"
- board text added: "1"
- board text added: "10"
- board text added: "11"
- board text added: "14"
- board text added: "15"
- board text added: "17"
- board text added: "18"
- board text added: "2"
- board text added: "22"
- board text added: "23"
- board text added: "24"
- board text added: "25"
- board text added: "27"
- board text added: "3"
- board text added: "3V3"
- board text added: "4"
- board text added: "5"
- board text added: "5V"
- board text added: "7"
- board text added: "8"
- board text added: "9"
- board text added: "CLK"
- board text added: "DAT"
- board text added: "GND"
- board text added: "IO:"
- board text added: "ISCP"
- board text added: "MCLR"
- board text added: "PI"
- board text added: "["
- board text added: "nc"
- board text removed: "RASPBERRY-PI 40-PIN ADDON BOARD VIEW FROM TOP NOTE: P1 SHOULD BE FITTED ON THE REVERSE OF THE BOARD ADD EDGE CUTS FROM CAMERA AND DISPLAY PORTS AS REQUIRED"

Commit message: version-e
Parts:
- C1: footprint Capacitor_THT:C_Disc_D3.8mm_W2.6mm_P2.50mm -> Capacitor_THT:C_Disc_D3.0mm_W2.0mm_P2.50mm
- moved C1 1.27 mm to (259.1, 120.8)
- moved D1 1.27 mm to (254.6, 106.8)
- moved R4 1.27 mm to (262.2, 110.6)
- moved R6 0.64 mm to (245.1, 127.1)
- moved SW1 0.64 mm to (248.3, 111.3)
- moved R1 0.63 mm to (233.0, 141.7)
- moved R5 0.63 mm to (241.9, 125.9)
Connections:
- J22 pad 10: +5V -> +3V3
- J22 pad 11: +5V -> +3V3
- J22 pad 12: +5V -> +3V3
- J22 pad 13: +5V -> +3V3
- J22 pad 7: +5V -> Net-(J22-Pad7)
- J22 pad 8: +5V -> +3V3
- J22 pad 9: +5V -> +3V3
Routing:
- net +3V3: track 33.2 -> 62.7 mm
- net +5V: track 83.0 -> 65.2 mm
- net +5VP: track 84.7 -> 82.5 mm
- net /DAT: track 26.5 -> 24.8 mm
- net /MCLR: track 20.6 -> 19.4 mm
- net /CLK: track 22.9 -> 21.9 mm
- net /IO1: track 6.82 -> 7.65 mm
- net Net-(R3-Pad2): track 10.3 -> 9.67 mm

Commit message: version-f (F.Cu filled, B.SilkS labels)
Routing:
- added copper zone on F.Cu, net GND
Other:
- board text added: "Rev F"
- board text added: "https://github.com/bablokb/pi-pic-proto-hat"
Changed lines of the file:
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@@
-(kicad_pcb (version 20171130) (host pcbnew 5.1.5+dfsg1-2~bpo10+1)
+(kicad_pcb (version 20171130) (host pcbnew 5.1.5-5.1.5)
   (general
     (thickness 1.6)
-    (drawings 64)
+    (drawings 70)
     (tracks 191)
     (zones 0)
@@
     (0 F.Cu signal)
     (31 B.Cu signal)
-    (32 B.Adhes user)
-    (33 F.Adhes user)
-    (34 B.Paste user)
-    (35 F.Paste user)
-    (36 B.SilkS user)
+    (32 B.Adhes user hide)
+    (33 F.Adhes user hide)
+    (34 B.Paste user hide)
+    (35 F.Paste user hide)
+    (36 B.SilkS user hide)
     (37 F.SilkS user)
-    (38 B.Mask user)
-    (39 F.Mask user)
-    (40 Dwgs.User user)
-    (41 Cmts.User user)
-    (42 Eco1.User user)
-    (43 Eco2.User user)
-    (44 Edge.Cuts user)
-    (45 Margin user)
-    (46 B.CrtYd user)
-    (47 F.CrtYd user)
+    (38 B.Mask user hide)
+    (39 F.Mask user hide)
+    (40 Dwgs.User user hide)
+    (41 Cmts.User user hide)
+    (42 Eco1.User user hide)
+    (43 Eco2.User user hide)
+    (44 Edge.Cuts user hide)
+    (45 Margin user hide)
+    (46 B.CrtYd user hide)
+    (47 F.CrtYd user hide)
   )
   (setup
-    (last_trace_width 0.8)
+    (last_trace_width 0.2)
     (user_trace_width 0.4)
     (user_trace_width 0.6)
@@
     (descr "Through hole straight pin header, 1x13, 2.54mm pitch, single row")
     (tags "Through hole pin header THT 1x13 2.54mm single row")
-    (fp_text reference J22 (at 0 -2.33 90) (layer F.SilkS)
+    (fp_text reference J22 (at 0 -2.33 90) (layer F.SilkS) hide
       (effects (font (size 1 1) (thickness 0.15)))
     )
@@
     )
   )
+  (gr_line (start 203.7084 105.042) (end 217.4498 104.8642) (layer F.SilkS) (width 0.15))
+  (gr_line (start 235.5346 104.8134) (end 220.7772 104.8388) (layer F.SilkS) (width 0.15))
+  (gr_line (start 203.7084 105.042) (end 202.6162 105.5246) (layer F.SilkS) (width 0.15))
+  (gr_line (start 235.56 104.8642) (end 235.9918 105.1944) (layer F.SilkS) (width 0.15))
+  (gr_text +5V (at 201.8034 107.0232 90) (layer F.SilkS)
+    (effects (font (size 1 1) (thickness 0.15)))
+  )
+  (gr_text "Rev F" (at 208.7122 148.0442) (layer B.SilkS)
+    (effects (font (size 1 1) (thickness 0.15)) (justify mirror))
+  )
+  (gr_text https://github.com/bablokb/pi-pic-proto-hat (at 240.1574 145.174) (layer B.SilkS)
+    (effects (font (size 1 1) (thickness 0.15)) (justify mirror))
+  )
   (gr_text [ (at 205.08 139.84) (layer F.SilkS)
     (effects (font (size 1 1) (thickness 0.15)))
@@
     (effects (font (size 1 1) (thickness 0.15)))
   )
-  (gr_text +3V3 (at 238.1 106.82 90) (layer F.SilkS)
-    (effects (font (size 1 1) (thickness 0.15)))
-  )
-  (gr_text +5V (at 236.83 106.82 90) (layer F.SilkS)
+  (gr_text +3V3 (at 236.957 107.0232 90) (layer F.SilkS)
     (effects (font (size 1 1) (thickness 0.15)))
   )
@@
       )
     )
+  )
+  (zone (net 3) (net_name GND) (layer F.Cu) (hatch edge 0.508)
+    (connect_pads (clearance 0.508))
+    (min_thickness 0.254)
+    (fill yes (arc_segments 32) (thermal_gap 0.508) (thermal_bridge_width 0.508))
+    (polygon
+      (pts
+        (xy 264.77 149.9746) (xy 200.0254 150) (xy 200.0762 94.0946) (xy 264.7954 94.0692)
+      )
+    )
