File: kicad/pi-pic-proto-hat/pipicproto.sch (KiCad schematic (older format))
At the start: 38 parts, among them J1 Conn_01x02_Male, J10 Conn_01x13_Male, J11 Conn_01x13_Male, J12 Conn_01x13_Male, J13 Conn_01x13_Male, J14 Conn_01x13_Male, J15 Conn_01x13_Male, J16 Conn_01x13_Male, J17 Conn_01x13_Male, J18 Conn_01x13_Male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

Commit message: version-b
Parts:
- removed JP1, JP2: Jumper_2_Open, symbol Jumper:Jumper_2_Open
- added J1, J4: Conn_01x02_Male, Connector_PinHeader_2.54mm:PinHeader_1x02_P2.54mm_Vertical, symbol Connector:Conn_01x02_Male
- C1: footprint (none) -> Capacitor_THT:C_Disc_D3.8mm_W2.6mm_P2.50mm
- D1: footprint (none) -> Diode_THT:D_A-405_P7.62mm_Horizontal
- J10: renamed from J8; footprint (none) -> Connector_PinHeader_2.54mm:PinHeader_1x13_P2.54mm_Vertical
- J11: renamed from J9; footprint (none) -> Connector_PinHeader_2.54mm:PinHeader_1x13_P2.54mm_Vertical
- J12: renamed from J10; footprint (none) -> Connector_PinHeader_2.54mm:PinHeader_1x13_P2.54mm_Vertical
- J13: renamed from J11; footprint (none) -> Connector_PinHeader_2.54mm:PinHeader_1x13_P2.54mm_Vertical
- J14: renamed from J12; footprint (none) -> Connector_PinHeader_2.54mm:PinHeader_1x13_P2.54mm_Vertical
- J15: renamed from J13; footprint (none) -> Connector_PinHeader_2.54mm:PinHeader_1x13_P2.54mm_Vertical
- J16: renamed from J14; footprint (none) -> Connector_PinHeader_2.54mm:PinHeader_1x13_P2.54mm_Vertical
- J17: renamed from J15; footprint (none) -> Connector_PinHeader_2.54mm:PinHeader_1x13_P2.54mm_Vertical
- J18: renamed from J16; footprint (none) -> Connector_PinHeader_2.54mm:PinHeader_1x13_P2.54mm_Vertical
- J19: renamed from J17; footprint (none) -> Connector_PinHeader_2.54mm:PinHeader_1x13_P2.54mm_Vertical
- J2: renamed from J1; footprint (none) -> Connector_Phoenix_MC:PhoenixContact_MC_1,5_2-G-3.81_1x02_P3.81mm_Horizontal
- J20: renamed from J18; footprint (none) -> Connector_PinHeader_2.54mm:PinHeader_1x13_P2.54mm_Vertical
- J21: renamed from J19; footprint (none) -> Connector_PinHeader_2.54mm:PinHeader_1x13_P2.54mm_Vertical
- J22: renamed from J20; footprint (none) -> Connector_PinHeader_2.54mm:PinHeader_1x13_P2.54mm_Vertical
- J3: renamed from J2; footprint (none) -> Connector_Phoenix_MC:PhoenixContact_MC_1,5_2-G-3.81_1x02_P3.81mm_Horizontal
- J5: renamed from J3; footprint (none) -> Connector_PinHeader_2.54mm:PinHeader_1x02_P2.54mm_Vertical
- J6: renamed from J4; footprint (none) -> Connector_BarrelJack:BarrelJack_CUI_PJ-102AH_Horizontal
- J7: renamed from J5; footprint (none) -> Connector_PinHeader_2.54mm:PinHeader_1x20_P2.54mm_Vertical
- J8: renamed from J6; footprint (none) -> Connector_PinHeader_2.54mm:PinHeader_1x06_P2.54mm_Vertical
- J9: renamed from J7; footprint (none) -> Connector_PinHeader_2.54mm:PinHeader_1x06_P2.54mm_Vertical
- R1, R2, R3, R4, R5, R6: footprint (none) -> Resistor_THT:R_Axial_DIN0207_L6.3mm_D2.5mm_P10.16mm_Horizontal
- SW1: footprint (none) -> Button_Switch_THT:SW_PUSH_6mm_H9.5mm
Connections:
- net +5V: now also J1.2 (Pin_2)
- net at J3.1 (Pin_1), Q1.2 (D): now also J1.1 (Pin_1)
- net at R2.2: now also J4.2 (Pin_2)
- net at J5.1 (Pin_1), J5.2 (Pin_2): now also J4.1 (Pin_1)

Commit message: version-e
Parts:
- C1: footprint Capacitor_THT:C_Disc_D3.8mm_W2.6mm_P2.50mm -> Capacitor_THT:C_Disc_D3.0mm_W2.0mm_P2.50mm
Connections:
- net +3V3: now also J22.10 (Pin_10), J22.11 (Pin_11), J22.12 (Pin_12), J22.13 (Pin_13), J22.8 (Pin_8), J22.9 (Pin_9)
- net +5V: no longer J22.10 (Pin_10), J22.11 (Pin_11), J22.12 (Pin_12), J22.13 (Pin_13), J22.7 (Pin_7), J22.8 (Pin_8), J22.9 (Pin_9)
- no-connect marks 157 -> 158
Changed lines of the file:
@@
-$EndComp
-$Comp
-L Connector:Conn_01x13_Male J22
-U 1 1 5E376781
-P 4300 5400
-F 0 "J22" H 4408 6089 50  0000 C CNN
-F 1 "Conn_01x13_Male" H 4408 6090 50  0001 C CNN
-F 2 "Connector_PinHeader_2.54mm:PinHeader_1x13_P2.54mm_Vertical" H 4300 5400 50  0001 C CNN
-F 3 "~" H 4300 5400 50  0001 C CNN
-	1    4300 5400
-	1    0    0    -1
 $EndComp
 $Comp
@@
 F 0 "C1" H 7615 3896 50  0000 L CNN
 F 1 "100n" H 7615 3805 50  0000 L CNN
-F 2 "Capacitor_THT:C_Disc_D3.8mm_W2.6mm_P2.50mm" H 7538 3700 50  0001 C CNN
+F 2 "Capacitor_THT:C_Disc_D3.0mm_W2.0mm_P2.50mm" H 7538 3700 50  0001 C CNN
 F 3 "~" H 7500 3850 50  0001 C CNN
 	1    7500 3850
@@
 Wire Wire Line
 	900  6000 900  6200
-Wire Wire Line
-	4500 4500 4500 4800
-Connection ~ 4500 4800
-Wire Wire Line
-	4500 4800 4500 4900
-Connection ~ 4500 4900
-Wire Wire Line
-	4500 4900 4500 5000
-Connection ~ 4500 5000
-Wire Wire Line
-	4500 5000 4500 5100
-Connection ~ 4500 5100
-Wire Wire Line
-	4500 5100 4500 5200
-Connection ~ 4500 5200
-Wire Wire Line
-	4500 5200 4500 5300
-Connection ~ 4500 5300
-Wire Wire Line
-	4500 5300 4500 5400
-Connection ~ 4500 5400
-Wire Wire Line
-	4500 5400 4500 5500
-Connection ~ 4500 5500
-Wire Wire Line
-	4500 5500 4500 5600
-Connection ~ 4500 5600
-Wire Wire Line
-	4500 5600 4500 5700
-Connection ~ 4500 5700
-Wire Wire Line
-	4500 5700 4500 5800
-Connection ~ 4500 5800
-Wire Wire Line
-	4500 5800 4500 5900
-Connection ~ 4500 5900
-Wire Wire Line
-	4500 5900 4500 6000
 NoConn ~ 4200 4800
 NoConn ~ 4200 4900
@@
 	8400 2600 8500 2600
 Connection ~ 8400 2600
+$Comp
+L Connector:Conn_01x13_Male J22
+U 1 1 5E376781
+P 4300 5400
+F 0 "J22" H 4408 6089 50  0000 C CNN
+F 1 "Conn_01x13_Male" H 4408 6090 50  0001 C CNN
+F 2 "Connector_PinHeader_2.54mm:PinHeader_1x13_P2.54mm_Vertical" H 4300 5400 50  0001 C CNN
+F 3 "~" H 4300 5400 50  0001 C CNN
+	1    4300 5400
+	1    0    0    -1
+$EndComp
+Wire Wire Line
+	4500 4500 4500 4800
+Connection ~ 4500 4800
+Wire Wire Line
+	4500 4800 4500 4900
+Connection ~ 4500 4900
+Wire Wire Line
+	4500 4900 4500 5000
+Connection ~ 4500 5000
+Wire Wire Line
+	4500 5000 4500 5100
+Connection ~ 4500 5100
+Wire Wire Line
+	4500 5100 4500 5200
+Connection ~ 4500 5200
+Wire Wire Line
+	4500 5200 4500 5300
+NoConn ~ 4500 5400
+$Comp
+L power:+3.3V #PWR0101
+U 1 1 5E48C144
+P 4750 4500
+F 0 "#PWR0101" H 4750 4350 50  0001 C CNN
+F 1 "+3.3V" H 4765 4673 50  0000 C CNN
+F 2 "" H 4750 4500 50  0001 C CNN
+F 3 "" H 4750 4500 50  0001 C CNN
+	1    4750 4500
+	1    0    0    -1
+$EndComp
+Wire Wire Line
+	4500 6000 4500 5900
+Connection ~ 4500 5600
+Wire Wire Line
+	4500 5600 4500 5500
+Connection ~ 4500 5700
+Wire Wire Line
+	4500 5700 4500 5600
+Connection ~ 4500 5800
+Wire Wire Line
+	4500 5800 4500 5700
+Connection ~ 4500 5900
+Wire Wire Line
+	4500 5900 4500 5800
+Wire Wire Line
+	4750 4500 4750 5500
+Wire Wire Line
+	4750 5500 4500 5500
+Connection ~ 4500 5500
 $EndSCHEMATC
