File: pi-pic-proto-hat.kicad/pipicproto.sch (KiCad schematic (older format))
At the start: 38 parts, among them J1 Conn_01x02_Male, J10 Conn_01x13_Male, J11 Conn_01x13_Male, J12 Conn_01x13_Male, J13 Conn_01x13_Male, J14 Conn_01x13_Male, J15 Conn_01x13_Male, J16 Conn_01x13_Male, J17 Conn_01x13_Male, J18 Conn_01x13_Male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

Commit message: added descriptive text
Other:
- note added: "5V to Pi\nPin 2/4"
- note added: "5V to ext.\nconnector J3 \n"
Changed lines of the file:
@@
 P 8500 2400
 F 0 "J5" V 8562 2444 50  0000 L CNN
-F 1 "Conn_01x02_Male" V 8653 2444 50  0000 L CNN
+F 1 "Conn_01x02_Male" V 8750 2150 50  0000 L CNN
 F 2 "Connector_PinHeader_2.54mm:PinHeader_1x02_P2.54mm_Vertical" H 8500 2400 50  0001 C CNN
 F 3 "~" H 8500 2400 50  0001 C CNN
@@
 P 7700 2400
 F 0 "J4" V 7762 2444 50  0000 L CNN
-F 1 "Conn_01x02_Male" V 7853 2444 50  0000 L CNN
+F 1 "Conn_01x02_Male" V 7950 2100 50  0000 L CNN
 F 2 "Connector_PinHeader_2.54mm:PinHeader_1x02_P2.54mm_Vertical" H 7700 2400 50  0001 C CNN
 F 3 "~" H 7700 2400 50  0001 C CNN
@@
 	4750 5500 4500 5500
 Connection ~ 4500 5500
+Text Notes 5200 850  2    50   ~ 0
+5V to Pi\nPin 2/4
+Text Notes 7850 1450 0    50   ~ 0
+5V to ext.\nconnector J3 \n
 $EndSCHEMATC

Commit message: V2.01: removed J4/J5/prototyping area
Parts:
- removed J11, J12, J13, J14, J15, J16, J17, J18, J19, J20, J21: Conn_01x13_Male, Connector_PinHeader_2.54mm:PinHeader_1x13_P2.54mm_Vertical, symbol Connector:Conn_01x13_Male
- removed J4, J5: Conn_01x02_Male, Connector_PinHeader_2.54mm:PinHeader_1x02_P2.54mm_Vertical, symbol Connector:Conn_01x02_Male
Connections:
- wire segments 176 -> 172
- no-connect marks 158 -> 29

Commit message: V2.02: connect GP0/GP1 directly to the Pi (add voltage-divider for GP1)
Parts:
- added R7: 6.2k, symbol Device:R
- added R8: 12k, symbol Device:R
- J9: value Conn_01x06_Male -> Conn_01x02_Male; footprint Connector_PinHeader_2.54mm:PinHeader_1x06_P2.54mm_Vertical -> Connector_PinHeader_2.54mm:PinHeader_1x02_P2.54mm_Vertical; symbol Connector:Conn_01x06_Male -> Connector:Conn_01x02_Male
Connections:
- net labels added: GPIO7(SPI0_CE_1), GPIO8(SPI0_CE_0)
- net labels removed: GPIO7(SPI1_CE_N), GPIO8(SPI0_CE_N), IO0, IO1, IO2, IO4, IO5
- wire segments 172 -> 169
- no-connect marks 29 -> 12
Other:
- note added: "GP2"
- note added: "GP4"
- note added: "PIC->Pi (gpio-shutdown)"
- note added: "Pi->PIC (gpio-poweroff)"
- moved on the sheet: J22
Changed lines of the file:
@@
 Title "PI PIC Prototyping Area"
 Date "2020-06-22"
-Rev "2.01"
+Rev "2.02"
 Comp "Bernhard Bablok, Lothar Hiller"
 Comment1 "https://github.com/bablokb/pi-pic-proto-hat"
@@
 ID_SC
 Text Label 3950 2300 2    50   ~ 0
-GPIO7(SPI1_CE_N)
+GPIO7(SPI0_CE_1)
 Text Label 3950 2200 2    50   ~ 0
-GPIO8(SPI0_CE_N)
+GPIO8(SPI0_CE_0)
 Text Label 3950 2100 2    50   ~ 0
 GPIO25(GEN6)
@@
 $EndComp
 $Comp
-L Connector:Conn_01x06_Male J9
+L Connector:Conn_01x02_Male J9
 U 1 1 5E2FB733
-P 10200 4500
-F 0 "J9" H 10150 4000 50  0000 R CNN
-F 1 "Conn_01x06_Male" H 10400 4100 50  0000 R CNN
-F 2 "Connector_PinHeader_2.54mm:PinHeader_1x06_P2.54mm_Vertical" H 10200 4500 50  0001 C CNN
-F 3 "~" H 10200 4500 50  0001 C CNN
-	1    10200 4500
-	-1   0    0    1
+P 9200 4250
+F 0 "J9" V 9250 4000 50  0000 R CNN
+F 1 "Conn_01x02_Male" V 9350 4000 50  0000 R CNN
+F 2 "Connector_PinHeader_2.54mm:PinHeader_1x02_P2.54mm_Vertical" H 9200 4250 50  0001 C CNN
+F 3 "~" H 9200 4250 50  0001 C CNN
+	1    9200 4250
+	0    -1   1    0
 $EndComp
 $Comp
@@
 L power:+5V #PWR015
 U 1 1 5E38E7EF
-P 4500 4500
-F 0 "#PWR015" H 4500 4350 50  0001 C CNN
-F 1 "+5V" H 4515 4673 50  0000 C CNN
-F 2 "" H 4500 4500 50  0001 C CNN
-F 3 "" H 4500 4500 50  0001 C CNN
-	1    4500 4500
+P 1450 4950
+F 0 "#PWR015" H 1450 4800 50  0001 C CNN
+F 1 "+5V" H 1465 5123 50  0000 C CNN
+F 2 "" H 1450 4950 50  0001 C CNN
+F 3 "" H 1450 4950 50  0001 C CNN
+	1    1450 4950
 	1    0    0    -1
 $EndComp
@@
 GPIO11(SPI0_SCK)
 Text Label 3600 4500 1    50   ~ 0
-GPIO8(SPI0_CE_N)
+GPIO8(SPI0_CE_0)
 Text Label 3700 4500 1    50   ~ 0
-GPIO7(SPI1_CE_N)
+GPIO7(SPI0_CE_1)
 $Comp
 L power:+5VP #PWR03
@@
 $EndComp
 Wire Wire Line
-	10000 4700 9650 4700
-Wire Wire Line
-	9650 4700 9650 6250
-Wire Wire Line
-	9650 6250 6400 6250
-Wire Wire Line
-	6400 6250 6400 5150
-Wire Wire Line
-	10000 4600 9500 4600
-Wire Wire Line
-	9500 4600 9500 6000
-Wire Wire Line
-	9500 6000 6800 6000
-Wire Wire Line
-	6800 6000 6800 5150
-Wire Wire Line
-	10000 4500 9350 4500
-Wire Wire Line
-	9350 4500 9350 5750
-Wire Wire Line
-	9350 5750 7250 5750
-Wire Wire Line
 	7250 5750 7250 4700
 Wire Wire Line
@@
 Wire Wire Line
 	7400 4500 6400 4500
-Wire Wire Line
-	7400 4600 6800 4600
 Wire Wire Line
 	6400 4850 6400 4500
 Connection ~ 6400 4500
-Wire Wire Line
-	6400 4500 5600 4500
 Wire Wire Line
 	6800 4850 6800 4600
@@
 Wire Wire Line
 	8600 4600 9200 4600
-Wire Wire Line
-	9200 4600 9200 4300
-Wire Wire Line
-	9200 4300 10000 4300
-Text Notes 9850 4950 0    50   ~ 0
+Text Notes 9150 3900 0    50   ~ 0
 PIC_GPIO
-Text Label 9700 4200 0    50   ~ 0
-IO5
-Text Label 9700 4300 0    50   ~ 0
-IO4
-Text Label 9700 4500 0    50   ~ 0
-IO2
-Text Label 9700 4600 0    50   ~ 0
-IO1
-Text Label 9700 4700 0    50   ~ 0
-IO0
-NoConn ~ 10000 4400
 NoConn ~ 5600 4700
 Text Notes 5400 4850 0    50   ~ 0
@@
 NoConn ~ 3950 2400
 NoConn ~ 3950 2600
-NoConn ~ 3950 2800
 NoConn ~ 3950 2900
 NoConn ~ 3950 3000
@@
 NoConn ~ 1250 2700
 NoConn ~ 1250 2800
-NoConn ~ 1250 2900
 Wire Wire Line
 	900  4800 900  4900
@@
 Wire Wire Line
 	900  6000 900  6200
-NoConn ~ 4200 4800
-NoConn ~ 4200 4900
-NoConn ~ 4200 5000
-NoConn ~ 4200 5100
-NoConn ~ 4200 5200
-NoConn ~ 4200 5300
-NoConn ~ 4200 5400
-NoConn ~ 4200 5500
-NoConn ~ 4200 5600
-NoConn ~ 4200 5700
-NoConn ~ 4200 5800
-NoConn ~ 4200 5900
-NoConn ~ 4200 6000
 Wire Wire Line
 	8000 5200 8000 5400
@@
 L Connector:Conn_01x13_Male J22
 U 1 1 5E376781
-P 4300 5400
-F 0 "J22" H 4408 6089 50  0000 C CNN
-F 1 "Conn_01x13_Male" H 4408 6090 50  0001 C CNN
-F 2 "Connector_PinHeader_2.54mm:PinHeader_1x13_P2.54mm_Vertical" H 4300 5400 50  0001 C CNN
-F 3 "~" H 4300 5400 50  0001 C CNN
-	1    4300 5400
-	1    0    0    -1
-$EndComp
-Wire Wire Line
-	4500 4500 4500 4800
-Connection ~ 4500 4800
-Wire Wire Line
-	4500 4800 4500 4900
-Connection ~ 4500 4900
-Wire Wire Line
-	4500 4900 4500 5000
-Connection ~ 4500 5000
-Wire Wire Line
-	4500 5000 4500 5100
-Connection ~ 4500 5100
-Wire Wire Line
-	4500 5100 4500 5200
-Connection ~ 4500 5200
-Wire Wire Line
-	4500 5200 4500 5300
-NoConn ~ 4500 5400
+P 1250 5850
+F 0 "J22" H 1358 6539 50  0000 C CNN
+F 1 "Conn_01x13_Male" H 1358 6540 50  0001 C CNN
+F 2 "Connector_PinHeader_2.54mm:PinHeader_1x13_P2.54mm_Vertical" H 1250 5850 50  0001 C CNN
+F 3 "~" H 1250 5850 50  0001 C CNN
+	1    1250 5850
+	1    0    0    -1
+$EndComp
+Wire Wire Line
+	1450 4950 1450 5250
+Connection ~ 1450 5250
+Wire Wire Line
+	1450 5250 1450 5350
+Connection ~ 1450 5350
+Wire Wire Line
+	1450 5350 1450 5450
+Connection ~ 1450 5450
+Wire Wire Line
+	1450 5450 1450 5550
+Connection ~ 1450 5550
+Wire Wire Line
+	1450 5550 1450 5650
+Connection ~ 1450 5650
+Wire Wire Line
+	1450 5650 1450 5750
+NoConn ~ 1450 5850
 $Comp
 L power:+3.3V #PWR0101
 U 1 1 5E48C144
-P 4750 4500
-F 0 "#PWR0101" H 4750 4350 50  0001 C CNN
-F 1 "+3.3V" H 4765 4673 50  0000 C CNN
-F 2 "" H 4750 4500 50  0001 C CNN
-F 3 "" H 4750 4500 50  0001 C CNN
-	1    4750 4500
-	1    0    0    -1
-$EndComp
-Wire Wire Line
-	4500 6000 4500 5900
-Connection ~ 4500 5600
-Wire Wire Line
-	4500 5600 4500 5500
-Connection ~ 4500 5700
-Wire Wire Line
-	4500 5700 4500 5600
-Connection ~ 4500 5800
-Wire Wire Line
-	4500 5800 4500 5700
-Connection ~ 4500 5900
-Wire Wire Line
-	4500 5900 4500 5800
-Wire Wire Line
-	4750 4500 4750 5500
-Wire Wire Line
-	4750 5500 4500 5500
-Connection ~ 4500 5500
+P 1700 4950
+F 0 "#PWR0101" H 1700 4800 50  0001 C CNN
+F 1 "+3.3V" H 1715 5123 50  0000 C CNN
+F 2 "" H 1700 4950 50  0001 C CNN
+F 3 "" H 1700 4950 50  0001 C CNN
+	1    1700 4950
+	1    0    0    -1
+$EndComp
+Wire Wire Line
+	1450 6450 1450 6350
+Connection ~ 1450 6050
+Wire Wire Line
+	1450 6050 1450 5950
+Connection ~ 1450 6150
+Wire Wire Line
+	1450 6150 1450 6050
+Connection ~ 1450 6250
+Wire Wire Line
+	1450 6250 1450 6150
+Connection ~ 1450 6350
+Wire Wire Line
+	1450 6350 1450 6250
+Wire Wire Line
+	1700 4950 1700 5950
+Wire Wire Line
+	1700 5950 1450 5950
+Connection ~ 1450 5950
 Text Notes 5200 850  2    50   ~ 0
 5V to Pi\nPin 2/4
 Text Notes 7850 1450 0    50   ~ 0
 5V to ext.\nconnector J3 \n
-NoConn ~ 10000 4200
 Wire Wire Line
 	8600 4700 8950 4700
@@
 Wire Wire Line
 	8950 2400 7300 2400
+Text Label 5850 5300 2    50   ~ 0
+GPIO16
+Text Label 5250 5650 2    50   ~ 0
+GPIO26
+$Comp
+L Device:R R7
+U 1 1 5EF5E7F1
+P 5850 5650
+F 0 "R7" V 5643 5650 50  0000 C CNN
+F 1 "6.2k" V 5734 5650 50  0000 C CNN
+F 2 "" V 5780 5650 50  0001 C CNN
+F 3 "~" H 5850 5650 50  0001 C CNN
+	1    5850 5650
+	0    1    1    0
+$EndComp
+$Comp
+L Device:R R8
+U 1 1 5EF5EC98
+P 5500 6000
+F 0 "R8" H 5570 6046 50  0000 L CNN
+F 1 "12k" H 5570 5955 50  0000 L CNN
+F 2 "" V 5430 6000 50  0001 C CNN
+F 3 "~" H 5500 6000 50  0001 C CNN
+	1    5500 6000
+	1    0    0    -1
+$EndComp
+$Comp
+L power:GND #PWR0102
+U 1 1 5EF66E1A
+P 5500 6150
+F 0 "#PWR0102" H 5500 5900 50  0001 C CNN
+F 1 "GND" H 5505 5977 50  0000 C CNN
+F 2 "" H 5500 6150 50  0001 C CNN
+F 3 "" H 5500 6150 50  0001 C CNN
+	1    5500 6150
+	1    0    0    -1
+$EndComp
+Wire Wire Line
+	5700 5650 5500 5650
+Wire Wire Line
+	5500 5850 5500 5650
+Connection ~ 5500 5650
+Wire Wire Line
+	5500 5650 5250 5650
+Text Notes 5100 5200 0    50   ~ 0
+Pi->PIC (gpio-poweroff)
+Text Notes 4450 5550 0    50   ~ 0
+PIC->Pi (gpio-shutdown)
+Wire Wire Line
+	5600 4500 6400 4500
+Wire Wire Line
+	6400 5150 6400 5300
+Wire Wire Line
+	5850 5300 6400 5300
+Wire Wire Line
+	6800 4600 7400 4600
+Wire Wire Line
+	6800 5150 6800 5650
+Wire Wire Line
+	6800 5650 6000 5650
+Wire Wire Line
+	9200 4600 9200 4450
+Wire Wire Line
+	7250 5750 9300 5750
+Wire Wire Line
+	9300 5750 9300 4450
+Text Notes 9200 4150 1    50   ~ 0
+GP4
+Text Notes 9350 4150 1    50   ~ 0
+GP2
 $EndSCHEMATC

Commit message: V2.03: removed reset-button, pullup, bat85
Parts:
- removed D1: D_Schottky, Diode_THT:D_A-405_P7.62mm_Horizontal, symbol Device:D_Schottky
- removed R3: 1k, Resistor_THT:R_Axial_DIN0207_L6.3mm_D2.5mm_P10.16mm_Horizontal, symbol Device:R
- removed R4: 22k, Resistor_THT:R_Axial_DIN0207_L6.3mm_D2.5mm_P10.16mm_Horizontal, symbol Device:R
- removed SW1: SW_Push, Button_Switch_THT:SW_PUSH_6mm_H9.5mm, symbol Switch:SW_Push
- R7, R8: footprint (none) -> Resistor_THT:R_Axial_DIN0207_L6.3mm_D2.5mm_P10.16mm_Horizontal
Connections:
- wire segments 169 -> 162
Changed lines of the file:
@@
 Title "PI PIC Prototyping Area"
 Date "2020-06-22"
-Rev "2.02"
+Rev "2.03"
 Comp "Bernhard Bablok, Lothar Hiller"
 Comment1 "https://github.com/bablokb/pi-pic-proto-hat"
@@
 $EndComp
 $Comp
-L Device:D_Schottky D1
-U 1 1 5E304BE1
-P 6400 3600
-F 0 "D1" H 6400 3816 50  0000 C CNN
-F 1 "D_Schottky" H 6400 3725 50  0000 C CNN
-F 2 "Diode_THT:D_A-405_P7.62mm_Horizontal" H 6400 3600 50  0001 C CNN
-F 3 "~" H 6400 3600 50  0001 C CNN
-	1    6400 3600
-	1    0    0    -1
-$EndComp
-$Comp
-L Device:R R4
-U 1 1 5E3051FC
-P 5750 3600
-F 0 "R4" V 5950 3600 50  0000 L CNN
-F 1 "22k" V 5850 3550 50  0000 L CNN
-F 2 "Resistor_THT:R_Axial_DIN0207_L6.3mm_D2.5mm_P10.16mm_Horizontal" V 5680 3600 50  0001 C CNN
-F 3 "~" H 5750 3600 50  0001 C CNN
-	1    5750 3600
-	0    -1   -1   0
-$EndComp
-$Comp
-L Switch:SW_Push SW1
-U 1 1 5E30C057
-P 6400 3200
-F 0 "SW1" H 6400 3485 50  0000 C CNN
-F 1 "SW_Push" H 6400 3394 50  0000 C CNN
-F 2 "Button_Switch_THT:SW_PUSH_6mm_H9.5mm" H 6400 3400 50  0001 C CNN
-F 3 "~" H 6400 3400 50  0001 C CNN
-	1    6400 3200
-	1    0    0    -1
-$EndComp
-$Comp
 L Device:R R6
 U 1 1 5E3133D0
@@
 F 3 "" H 6000 4400 50  0001 C CNN
 	1    6000 4400
-	0    -1   -1   0
-$EndComp
-$Comp
-L power:GND #PWR09
-U 1 1 5E340737
-P 6800 3200
-F 0 "#PWR09" H 6800 2950 50  0001 C CNN
-F 1 "GND" V 6805 3072 50  0000 R CNN
-F 2 "" H 6800 3200 50  0001 C CNN
-F 3 "" H 6800 3200 50  0001 C CNN
-	1    6800 3200
 	0    -1   -1   0
 $EndComp
@@
 Wire Wire Line
 	5600 3750 5600 4200
-$Comp
-L Device:R R3
-U 1 1 5E3838F5
-P 5750 3200
-F 0 "R3" V 5950 3150 50  0000 L CNN
-F 1 "1k" V 5850 3150 50  0000 L CNN
-F 2 "Resistor_THT:R_Axial_DIN0207_L6.3mm_D2.5mm_P10.16mm_Horizontal" V 5680 3200 50  0001 C CNN
-F 3 "~" H 5750 3200 50  0001 C CNN
-	1    5750 3200
-	0    -1   -1   0
-$EndComp
-Wire Wire Line
-	5600 3600 5600 3750
-Connection ~ 5600 3750
-Wire Wire Line
-	5600 3200 5600 3600
-Connection ~ 5600 3600
-Wire Wire Line
-	5900 3200 6200 3200
-Wire Wire Line
-	6600 3200 6800 3200
-Wire Wire Line
-	5900 3600 6250 3600
-Wire Wire Line
-	6550 3600 7250 3600
-Wire Wire Line
-	7250 3600 7250 4000
-Connection ~ 7250 4000
 Wire Wire Line
 	8750 3750 5600 3750
@@
 F 0 "R7" V 5643 5650 50  0000 C CNN
 F 1 "6.2k" V 5734 5650 50  0000 C CNN
-F 2 "" V 5780 5650 50  0001 C CNN
+F 2 "Resistor_THT:R_Axial_DIN0207_L6.3mm_D2.5mm_P10.16mm_Horizontal" V 5780 5650 50  0001 C CNN
 F 3 "~" H 5850 5650 50  0001 C CNN
 	1    5850 5650
@@
 F 0 "R8" H 5570 6046 50  0000 L CNN
 F 1 "12k" H 5570 5955 50  0000 L CNN
-F 2 "" V 5430 6000 50  0001 C CNN
+F 2 "Resistor_THT:R_Axial_DIN0207_L6.3mm_D2.5mm_P10.16mm_Horizontal" V 5430 6000 50  0001 C CNN
 F 3 "~" H 5500 6000 50  0001 C CNN
 	1    5500 6000
